File: kicad/bottom/bottom.kicad_sch (KiCad schematic)
At the start: 37 parts, among them J1 Conn_01x15_Socket

Commit message: removed scottokeebs kicad files, updated the mounting holes to use m2.5 instead of m2, added m2.5 footprints to each pcbs footprint library
Parts:
- H1, H2, H3, H4: footprint MountingHole:MountingHole_2.5mm_Pad -> Bottom-Footprints:MountingHole_2.5mm_Pad
Changed lines of the file:
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@@
 			)
 		)
-		(property "Footprint" "MountingHole:MountingHole_2.5mm_Pad"
+		(property "Footprint" "Bottom-Footprints:MountingHole_2.5mm_Pad"
 			(at 182.88 101.6 0)
 			(effects
@@
 			)
 		)
-		(property "Footprint" "MountingHole:MountingHole_2.5mm_Pad"
+		(property "Footprint" "Bottom-Footprints:MountingHole_2.5mm_Pad"
 			(at 191.77 101.6 0)
 			(effects
@@
 			)
 		)
-		(property "Footprint" "MountingHole:MountingHole_2.5mm_Pad"
+		(property "Footprint" "Bottom-Footprints:MountingHole_2.5mm_Pad"
 			(at 191.77 114.3 0)
 			(effects
@@
 			)
 		)
-		(property "Footprint" "MountingHole:MountingHole_2.5mm_Pad"
+		(property "Footprint" "Bottom-Footprints:MountingHole_2.5mm_Pad"
 			(at 182.88 114.3 0)
 			(effects
