File: kicad/top/top.kicad_sch (KiCad schematic)
At the start: 32 parts, among them J1 OLED_128x32, J2 Conn_01x15, SW1 SLW-864574-5A-RA-N-D, SW2 RotaryEncoder_Switch

Commit message: removed scottokeebs kicad files, updated the mounting holes to use m2.5 instead of m2, added m2.5 footprints to each pcbs footprint library
Parts:
- H1, H2, H3, H4: footprint MountingHole:MountingHole_2.5mm_Pad -> Top-Footprints:MountingHole_2.5mm_Pad
Changed lines of the file:
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@@
 			)
 		)
-		(property "Footprint" "MountingHole:MountingHole_2.5mm_Pad"
+		(property "Footprint" "Top-Footprints:MountingHole_2.5mm_Pad"
 			(at 190.5 59.69 0)
 			(effects
@@
 			)
 		)
-		(property "Footprint" "MountingHole:MountingHole_2.5mm_Pad"
+		(property "Footprint" "Top-Footprints:MountingHole_2.5mm_Pad"
 			(at 205.74 72.39 0)
 			(effects
@@
 			)
 		)
-		(property "Footprint" "MountingHole:MountingHole_2.5mm_Pad"
+		(property "Footprint" "Top-Footprints:MountingHole_2.5mm_Pad"
 			(at 190.5 72.39 0)
 			(effects
@@
 			)
 		)
-		(property "Footprint" "MountingHole:MountingHole_2.5mm_Pad"
+		(property "Footprint" "Top-Footprints:MountingHole_2.5mm_Pad"
 			(at 205.74 59.69 0)
 			(effects
